File: spark-inducer/spark-inducer.kicad_pcb (KiCad board)
At the start: 2 copper layers, 233.3 x 128.5 mm, 84 parts, among them J1 POWER IN, J10 IO_A_1, J11 IO_A_3, J12 IO_A_2, J13 IO_A_4, J14 IO_B_1, J15 IO_B_3, J16 IO_B_2, J17 IO_B_4, J18 REF_SELECT, J19 POWER_A_1, J2 IO1, J20 POWER_A_2, J21 POWER_A_3, J22 POWER_A_4, J23 POWER_B_1, J24 POWER_B_2, J25 POWER_B_3, J26 POWER_B_4, J3 IO2, J4 IO3, J5 IO4, J6 IO5, J7 IO6, J8 OUT1, J9 OUT2, SW1 SWITCH, U1 TL072B, U2 TL072B, U3 TL431BD, U4 L78LXX, U5 LM4040, U6 REF50XX

Commit message: Update to KiCad 6
Parts:
- U3: value TL431BD -> TL431B
- moved Logo 14.5 mm to (197.7, 162.0)
- renumbered REF** to BREADBOARD_BOTTOM, REF** to BREADBOARD_TOP, REF** to SCREW_PANEL_BL, REF** to SCREW_PANEL_BR, REF** to SCREW_PANEL_TL, REF** to SCREW_PANEL_TR, REF** to SCREW_SWITCH_BOTTOM, REF** to SCREW_SWITCH_TOP
Connections:
- U6 pad 1: Net-(U6-Pad1) -> unconnected-(U6-Pad1)
- U6 pad 3: Net-(U6-Pad3) -> unconnected-(U6-Pad3)
- U6 pad 5: Net-(U6-Pad5) -> unconnected-(U6-Pad5)
- U6 pad 7: Net-(U6-Pad7) -> unconnected-(U6-Pad7)
- U6 pad 8: Net-(U6-Pad8) -> unconnected-(U6-Pad8)
Routing:
- net +12V: track 590.9 -> 593.9 mm
- net /IO_4_TN: track 36.5 -> 35.5 mm
- net /IO_5_TN: track 300.9 -> 300.2 mm
- net /IO_1_TN: track 82.1 -> 81.4 mm
- net /IO_1_T: track 72.1 -> 71.3 mm
- net -12V: track 430.8 -> 431.5 mm
Other:
- net class Default removed
- net class Power removed
- board text added: "+5V"
- board text added: "FUSE +12V"
- board text added: "FUSE +5V"
- board text added: "FUSE -12V"
- board text added: "RED STRIPE"
- board text added: "T"

Commit message: Update all footprints, use new custom footprints
Parts:
- removed G***: LOGO, Protorack2:TSKF_45x4mm
- removed SCREW_PANEL_BL, SCREW_PANEL_BR, SCREW_PANEL_TL, SCREW_PANEL_TR: Screw_ISO7380_M3x6, Protorack:Screw_ISO7380_M3x6
- removed SCREW_SWITCH_BOTTOM, SCREW_SWITCH_TOP: Screw_ISO4762_M2x6, Protorack:Screw_ISO4762_M2x6
- added H1: SCREW_SW_TOP, Protorack:Screw_ISO4762_M2x6, F.Cu at (56.2, 50.2)
- added H10: NUT_OUT1, Protorack:Nut_M6x2mm_Knurled, F.Cu at (41.7, 145.5)
- added H11: NUT_IO2, Protorack:Nut_M6x2mm_Knurled, F.Cu at (55.7, 85.5)
- added H12: NUT_IO4, Protorack:Nut_M6x2mm_Knurled, F.Cu at (55.7, 105.5)
- added H13: NUT_IO6, Protorack:Nut_M6x2mm_Knurled, F.Cu at (55.7, 125.5)
- added H14: NUT_OUT2, Protorack:Nut_M6x2mm_Knurled, F.Cu at (55.7, 145.5)
- added H15: NUT_POT_A, Protorack:Nut_M7x2mm_Black, F.Cu at (245.7, 58.5)
- added H16: NUT_POT_B, Protorack:Nut_M7x2mm_Black, F.Cu at (245.7, 85.5)
- added H17: NUT_POT_C, Protorack:Nut_M7x2mm_Black, F.Cu at (245.7, 112.5)
- added H18: NUT_POT_D, Protorack:Nut_M7x2mm_Black, F.Cu at (245.7, 139.5)
- added H19: WASHER_POT_A, Protorack:Washer_RV16AF_2mm_Tab, F.Cu at (245.7, 58.5)
- added H2: SCREW_SW_BOT, Protorack:Screw_ISO4762_M2x6, F.Cu at (56.2, 70.8)
- added H20: WASHER_POT_B, Protorack:Washer_RV16AF_2mm_Tab, F.Cu at (245.7, 85.5)
- added H21: WASHER_POT_C, Protorack:Washer_RV16AF_2mm_Tab, F.Cu at (245.7, 112.5)
- added H22: WASHER_POT_D, Protorack:Washer_RV16AF_2mm_Tab, F.Cu at (245.7, 139.5)
- added H3: SCREW_PANEL_TL, Protorack:Screw_ISO7380_M3x6, F.Cu at (38.2, 41.8)
- added H4: SCREW_PANEL_TR, Protorack:Screw_ISO7380_M3x6, F.Cu at (256.6, 41.8)
- added H5: SCREW_PANEL_BL, Protorack:Screw_ISO7380_M3x6, F.Cu at (38.2, 164.2)
- added H6: SCREW_PANEL_BR, Protorack:Screw_ISO7380_M3x6, F.Cu at (256.6, 164.2)
- added H7: NUT_IO1, Protorack:Nut_M6x2mm_Knurled, F.Cu at (41.7, 85.5)
- added H8: NUT_IO3, Protorack:Nut_M6x2mm_Knurled, F.Cu at (41.7, 105.5)
- added H9: NUT_IO5, Protorack:Nut_M6x2mm_Knurled, F.Cu at (41.7, 125.5)
- added REF**: TSKF_44x4mm, Protorack:TSKF_44x4mm, B.Cu at (147.3, 162.0)
- C5, C6, C7, C8: footprint Capacitor_SMD:C_1206_3216Metric_Pad1.42x1.75mm_HandSolder -> Capacitor_SMD:C_1206_3216Metric_Pad1.33x1.80mm_HandSolder
- J1: value POWER IN -> Eurorack_Power_Header; footprint Protorack:Samtec_HTST-108-01-T-DV -> Protorack:Eurorack_Power_Header_2x08_SMD_HandSolder
- J10, J11, J12, J13, J14, J15, J16, J17: footprint Protorack:Samtec_TSW-106-09-T-S-RA_Shortened_SurfaceMount -> Protorack:Samtec_TSW-106-09-T-S-RA_Shortened_SMD; moved to F.Cu
- J2, J3, J4, J5, J6, J7, J8, J9: footprint Protorack:QingPu_WQP-PJ376M_SurfaceMount -> Protorack:QingPu_WQP-WQP518MA-BM_SMD
- R10, R11: value 18k -> 33k 0.1%
- RV1, RV2, RV3, RV4: footprint Protorack:Alpha_RV16AF-20-15F_SurfaceMount_Nut_Knob -> Protorack:Alpha_RV16AF-10-17K_SMD_Slot
- SW1: footprint Protorack:CW_GF-161-3011_SurfaceMount -> Protorack:CW_GF-161-3011_SMD
- moved QRCode 5.00 mm to (240.7, 161.5)
- turned D6 to 180 degrees
- turned J1 to 180 degrees
- turned J10 to 180 degrees
- turned J11 to 0 degrees
- turned J12 to 180 degrees
- turned J13 to 0 degrees
- turned J14 to 180 degrees
- turned J15 to 0 degrees
- turned J16 to 180 degrees
- turned J17 to 0 degrees
- turned RV1 to -10 degrees
- turned RV2 to -10 degrees
- turned RV3 to -10 degrees
- turned RV4 to -10 degrees
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Routing:
- net unconnected-(J1-PadGATE): track 0.00 -> 8.89 mm
- net unconnected-(J1-PadCV): track 0.00 -> 8.89 mm
- net Net-(J1-Pad15): track 8.89 -> 0.00 mm
- net Net-(J1-Pad13): track 8.89 -> 0.00 mm
- net /POT_D_1: track 29.1 -> 25.5 mm
- net /POT_C_2: track 58.0 -> 54.7 mm
- net /POT_B_3: track 271.0 -> 274.2 mm
- net +5V: track 427.8 -> 430.9 mm
- net /POT_A_2: track 273.0 -> 270.3 mm
- net /POT_D_2: track 31.7 -> 29.0 mm
- net /POT_C_3: track 60.6 -> 58.2 mm
- net /POT_B_2: track 278.3 -> 280.6 mm
- net /POT_A_1: track 262.8 -> 260.7 mm
- net /POT_C_1: track 55.5 -> 53.4 mm
- net -12V: track 431.5 -> 433.3 mm
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Other:
- outline, holes or cut-outs redrawn
- board text added: "33k 0.1%"
