File: helper-jack/helper-jack.kicad_sch (KiCad schematic)
At the start: 4 parts, among them J1 S, J2 T, J3 TN, J4 WQP518MA-BM_Combined

Commit message: Update helper jack to KiCad 7, Adjust markings, jack footprint
Parts:
- J4: symbol Connector:AudioJack2_SwitchT -> Connector_Audio:AudioJack2_SwitchT
Changed lines of the file:
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@@
-(kicad_sch (version 20211123) (generator eeschema)
+(kicad_sch (version 20230121) (generator eeschema)
   (paper "A4")
   (wire (pts (xy 57.15 22.86) (xy 59.69 22.86))
-    (stroke (width 0) (type default) (color 0 0 0 0))
+    (stroke (width 0) (type default))
   )
   (wire (pts (xy 33.02 21.59) (xy 30.48 21.59))
-    (stroke (width 0) (type default) (color 0 0 0 0))
+    (stroke (width 0) (type default))
   )
   (wire (pts (xy 57.15 27.94) (xy 59.69 27.94))
-    (stroke (width 0) (type default) (color 0 0 0 0))
+    (stroke (width 0) (type default))
   )
   (wire (pts (xy 33.02 29.21) (xy 30.48 29.21))
-    (stroke (width 0) (type default) (color 0 0 0 0))
+    (stroke (width 0) (type default))
   )
   (wire (pts (xy 33.02 25.4) (xy 30.48 25.4))
-    (stroke (width 0) (type default) (color 0 0 0 0))
+    (stroke (width 0) (type default))
   )
   (wire (pts (xy 57.15 25.4) (xy 59.69 25.4))
-    (stroke (width 0) (type default) (color 0 0 0 0))
+    (stroke (width 0) (type default))
   )
-  (label "TN" (at 33.02 29.21 0)
+  (label "TN" (at 33.02 29.21 0) (fields_autoplaced)
     (effects (font (size 1.27 1.27)) (justify left bottom))
   )
-  (label "T" (at 33.02 25.4 0)
+  (label "T" (at 33.02 25.4 0) (fields_autoplaced)
     (effects (font (size 1.27 1.27)) (justify left bottom))
   )
-  (label "S" (at 33.02 21.59 0)
+  (label "S" (at 33.02 21.59 0) (fields_autoplaced)
     (effects (font (size 1.27 1.27)) (justify left bottom))
   )
-  (label "TN" (at 59.69 27.94 0)
+  (label "TN" (at 59.69 27.94 0) (fields_autoplaced)
     (effects (font (size 1.27 1.27)) (justify left bottom))
   )
-  (label "T" (at 59.69 25.4 0)
+  (label "T" (at 59.69 25.4 0) (fields_autoplaced)
     (effects (font (size 1.27 1.27)) (justify left bottom))
   )
-  (label "S" (at 59.69 22.86 0)
+  (label "S" (at 59.69 22.86 0) (fields_autoplaced)
     (effects (font (size 1.27 1.27)) (justify left bottom))
   )
   (symbol (lib_id "Connector_Generic:Conn_01x01") (at 25.4 25.4 0) (mirror y) (unit 1)
-    (in_bom yes) (on_board yes)
-    (property "Reference" "J2" (id 0) (at 21.59 25.4 0))
-    (property "Value" "T" (id 1) (at 17.78 25.4 0))
-    (property "Footprint" "TestPoint:TestPoint_THTPad_2.0x2.0mm_Drill1.0mm" (id 2) (at 25.4 25.4 0)
+    (in_bom yes) (on_board yes) (dnp no)
+    (property "Reference" "J2" (at 21.59 25.4 0)
+      (effects (font (size 1.27 1.27)))
+    )
+    (property "Value" "T" (at 17.78 25.4 0)
+      (effects (font (size 1.27 1.27)))
+    )
+    (property "Footprint" "TestPoint:TestPoint_THTPad_2.0x2.0mm_Drill1.0mm" (at 25.4 25.4 0)
       (effects (font (size 1.27 1.27)) hide)
     )
-    (property "Datasheet" "~" (id 3) (at 25.4 25.4 0)
+    (property "Datasheet" "~" (at 25.4 25.4 0)
       (effects (font (size 1.27 1.27)) hide)
     )
     (pin "1")
+    (instances
+      (project "helper-jack"
+        (path "/08402209-d3fd-42d4-8065-6a77e812c43c"
+          (reference "J2") (unit 1)
+        )
+      )
+    )
   )
   (symbol (lib_id "Connector_Generic:Conn_01x01") (at 25.4 21.59 0) (mirror y) (unit 1)
-    (in_bom yes) (on_board yes)
-    (property "Reference" "J1" (id 0) (at 21.59 21.59 0))
-    (property "Value" "S" (id 1) (at 17.78 21.59 0))
-    (property "Footprint" "TestPoint:TestPoint_THTPad_2.0x2.0mm_Drill1.0mm" (id 2) (at 25.4 21.59 0)
+    (in_bom yes) (on_board yes) (dnp no)
+    (property "Reference" "J1" (at 21.59 21.59 0)
+      (effects (font (size 1.27 1.27)))
+    )
+    (property "Value" "S" (at 17.78 21.59 0)
+      (effects (font (size 1.27 1.27)))
+    )
+    (property "Footprint" "TestPoint:TestPoint_THTPad_2.0x2.0mm_Drill1.0mm" (at 25.4 21.59 0)
       (effects (font (size 1.27 1.27)) hide)
     )
-    (property "Datasheet" "~" (id 3) (at 25.4 21.59 0)
+    (property "Datasheet" "~" (at 25.4 21.59 0)
       (effects (font (size 1.27 1.27)) hide)
     )
     (pin "1")
+    (instances
+      (project "helper-jack"
+        (path "/08402209-d3fd-42d4-8065-6a77e812c43c"
+          (reference "J1") (unit 1)
+        )
+      )
+    )
   )
-  (symbol (lib_id "Connector:AudioJack2_SwitchT") (at 52.07 25.4 0) (unit 1)
-    (in_bom yes) (on_board yes)
-    (property "Reference" "J4" (id 0) (at 52.07 16.51 0))
-    (property "Value" "WQP518MA-BM_Combined" (id 1) (at 52.07 19.05 0))
-    (property "Footprint" "Protorack:QingPu_WQP-WQP518MA-BM_Combined" (id 2) (at 52.07 25.4 0)
+  (symbol (lib_id "Connector_Audio:AudioJack2_SwitchT") (at 52.07 25.4 0) (unit 1)
+    (in_bom yes) (on_board yes) (dnp no)
+    (property "Reference" "J4" (at 52.07 16.51 0)
+      (effects (font (size 1.27 1.27)))
+    )
+    (property "Value" "WQP518MA-BM_Combined" (at 52.07 19.05 0)
+      (effects (font (size 1.27 1.27)))
+    )
+    (property "Footprint" "Protorack:QingPu_WQP-WQP518MA-BM_Combined" (at 52.07 25.4 0)
       (effects (font (size 1.27 1.27)) hide)
     )
-    (property "Datasheet" "~" (id 3) (at 52.07 25.4 0)
+    (property "Datasheet" "~" (at 52.07 25.4 0)
       (effects (font (size 1.27 1.27)) hide)
     )
@@
     (pin "T")
     (pin "TN")
+    (instances
+      (project "helper-jack"
+        (path "/08402209-d3fd-42d4-8065-6a77e812c43c"
+          (reference "J4") (unit 1)
+        )
+      )
+    )
   )
   (symbol (lib_id "Connector_Generic:Conn_01x01") (at 25.4 29.21 0) (mirror y) (unit 1)
-    (in_bom yes) (on_board yes)
-    (property "Reference" "J3" (id 0) (at 21.59 29.21 0))
-    (property "Value" "TN" (id 1) (at 17.78 29.21 0))
-    (property "Footprint" "TestPoint:TestPoint_THTPad_2.0x2.0mm_Drill1.0mm" (id 2) (at 25.4 29.21 0)
+    (in_bom yes) (on_board yes) (dnp no)
+    (property "Reference" "J3" (at 21.59 29.21 0)
+      (effects (font (size 1.27 1.27)))
+    )
+    (property "Value" "TN" (at 17.78 29.21 0)
+      (effects (font (size 1.27 1.27)))
+    )
+    (property "Footprint" "TestPoint:TestPoint_THTPad_2.0x2.0mm_Drill1.0mm" (at 25.4 29.21 0)
       (effects (font (size 1.27 1.27)) hide)
     )
-    (property "Datasheet" "~" (id 3) (at 25.4 29.21 0)
+    (property "Datasheet" "~" (at 25.4 29.21 0)
       (effects (font (size 1.27 1.27)) hide)
     )
     (pin "1")
+    (instances
+      (project "helper-jack"
+        (path "/08402209-d3fd-42d4-8065-6a77e812c43c"
+          (reference "J3") (unit 1)
+        )
+      )
+    )
   )
   (sheet_instances
     (path "/" (page "1"))
   )
-  (symbol_instances
-    (path "/584dd6f4-b2b6-4752-a0db-43c61228b55e"
-      (reference "J1") (unit 1) (value "S") (footprint "TestPoint:TestPoint_THTPad_2.0x2.0mm_Drill1.0mm")
-    )
-    (path "/21aebbca-77b7-4716-9e34-729899f8b713"
-      (reference "J2") (unit 1) (value "T") (footprint "TestPoint:TestPoint_THTPad_2.0x2.0mm_Drill1.0mm")
-    )
-    (path "/8aff7831-39c5-43f8-b21c-3814575054d2"
-      (reference "J3") (unit 1) (value "TN") (footprint "TestPoint:TestPoint_THTPad_2.0x2.0mm_Drill1.0mm")
-    )
-    (path "/70b8744a-7f56-4a6d-a71a-1de076f49081"
-      (reference "J4") (unit 1) (value "WQP518MA-BM_Combined") (footprint "Protorack:QingPu_WQP-WQP518MA-BM_Combined")
-    )
-  )
 )
