File: helper-switch/helper-switch.kicad_sch (KiCad schematic)
At the start: 7 parts, among them J1 +5V_IN, J2 +5V_OUT, J3 +12V_IN, J4 +12V_OUT, J5 -12V_IN, J6 -12V_OUT, SW1 POWER

Commit message: Update helper switch to KiCad 7, Adjust markings
Connections:
- net +12V_IN: now also SW1.6 (C); no longer SW1.5 (B)
- net +12V_OUT: now also SW1.5 (B); no longer SW1.6 (C)
- net +5V_IN: now also SW1.3 (C); no longer SW1.2 (B)
- net +5V_OUT: now also SW1.2 (B); no longer SW1.3 (C)
